Commit message: refactored to compile in humble

File: bot_description/urdf/chassis.urdf.xacro (robot description, xacro)
@@ -1,5 +1,5 @@
 <robot name="robopi"
-       xmlns:xacro="http://www.ros.org/wiki/xacro"
-       xmlns:xi="http://www.w3.org/2001/XInclude">
+    xmlns:xacro="http://www.ros.org/wiki/xacro"
+    xmlns:xi="http://www.w3.org/2001/XInclude">
     <xacro:property name="chassis_len" value=".19"/>
     <xacro:property name="chassis_width" value=".19"/>
@@ -9,5 +9,5 @@
             <origin rpy="-${PI/2} 0 ${PI/2}" xyz="0 0 0"/>
             <geometry>
-                <mesh filename="package://robopi/meshes/base_assembly.dae"/>
+                <mesh filename="package://bot_description/meshes/base_assembly.dae"/>
             </geometry>
         </visual>
@@ -15,5 +15,5 @@
             <origin rpy="-${PI/2} 0 0" xyz="0 0 0"/>
             <geometry>
-                <mesh filename="package://robopi/meshes/base_assembly.dae"/>
+                <mesh filename="package://bot_description/meshes/base_assembly.dae"/>
             </geometry>
         </collision>

File: bot_description/urdf/globals.urdf.xacro (robot description, xacro)
@@ -1,4 +1,5 @@
 <?xml version="1.0"?>
-<robot name="robopi" xmlns:xacro="http://www.ros.org/wiki/xacro">
+<robot name="robopi"
+    xmlns:xacro="http://www.ros.org/wiki/xacro">
     <!-- /////////////////////////////////////////////////////////////////-->
     <!-- Include materials-->
@@ -17,7 +18,5 @@
         <inertial>
             <mass value="${m}"/>
-            <inertia ixx="${m*(3*r*r+h*h)/12}"  ixy="0.0" ixz="0.0"
-                     iyy="${m*(3*r*r+h*h)/12}"  iyz= "0.0"
-                     izz="${m*r*r/2}"/>
+            <inertia ixx="${m*(3*r*r+h*h)/12}" ixy="0.0" ixz="0.0" iyy="${m*(3*r*r+h*h)/12}" iyz= "0.0" izz="${m*r*r/2}"/>
         </inertial>
     </xacro:macro>
@@ -26,7 +25,5 @@
         <inertial>
             <mass value="${mass}"/>
-            <inertia ixx="1.0" ixy="0.0"
-                     iyy="1.0" iyz="0.0"
-                     izz="1.0" ixz="0.0"/>
+            <inertia ixx="1.0" ixy="0.0" iyy="1.0" iyz="0.0" izz="1.0" ixz="0.0"/>
         </inertial>
     </xacro:macro>

File: bot_description/urdf/robopi.urdf.xacro (robot description, xacro)
@@ -1,5 +1,5 @@
-<robot name="robopi"
-       xmlns:xacro="http://www.ros.org/wiki/xacro"
-       xmlns:xi="http://www.w3.org/2001/XInclude">
+<robot name="bot"
+    xmlns:xacro="http://www.ros.org/wiki/xacro"
+    xmlns:xi="http://www.w3.org/2001/XInclude">
     <xacro:include filename="globals.urdf.xacro" />
     <xacro:include filename="chassis.urdf.xacro" />

File: bot_description/urdf/sonar.urdf.xacro (robot description, xacro)
@@ -1,5 +1,5 @@
 <robot name="robopi"
-       xmlns:xacro="http://www.ros.org/wiki/xacro"
-       xmlns:xi="http://www.w3.org/2001/XInclude">
+    xmlns:xacro="http://www.ros.org/wiki/xacro"
+    xmlns:xi="http://www.w3.org/2001/XInclude">
     <link name="sonar_front">
         <visual>
