Commit message: update xml, updated serial protocol

File: bot_description/urdf/wheels.urdf.xacro (robot description, xacro)
@@ -1,3 +1,3 @@
-<robot name="robopi"
+<robot name="bot"
   xmlns:xacro="http://www.ros.org/wiki/xacro"
   xmlns:xi="http://www.w3.org/2001/XInclude">
@@ -6,17 +6,18 @@
   <xacro:property name="wheel_height" value="0.11"/>
   <xacro:property name="wheel_mass" value=".2"/>
-  <xacro:macro name="Transmission_block" params="joint_name">
-    <transmission name="${joint_name}_trans">
-      <type>transmission_interface/SimpleTransmission</type>
-      <joint name="${joint_name}">
-        <hardwareInterface>PositionJointInterface</hardwareInterface>
-      </joint>
-      <actuator name="${joint_name}_motor">
-        <mechanicalReduction>1</mechanicalReduction>
-      </actuator>
-    </transmission>
-  </xacro:macro>
-  <xacro:macro name="wheel" params= "prefix suffix X Y Z">
-    <link name= "${prefix}_${suffix}_wheel">
+  <xacro:macro name="wheel" params= "prefix X Y Z">
+    <joint name="${prefix}_wheel_joint1" type= "fixed">
+      <parent link="${prefix}_wheel"/>
+      <child link= "${prefix}_wheel1"/>
+      <origin xyz="0 0 0" rpy="0 0 0"/>
+    </joint>
+    <joint name="${prefix}_wheel_joint" type="continuous">
+      <parent link= "base_link"/>
+      <child link= "${prefix}_wheel"/>
+      <origin xyz= "${0.062*X-0.058*Y} ${(chassis_len/2+0.02)*Z}  0.015" rpy="0 0 0"/>
+      <axis xyz="0 1 0"/>
+      <dynamics damping="0.0" friction="0.0"/>
+    </joint>
+    <link name= "${prefix}_wheel">
       <visual>
         <origin rpy= "${PI/2} 0 0" xyz= "0 0 0"/>
@@ -34,9 +35,9 @@
       <xacro:cylinder_inertia m="${wheel_mass}" r="${wheel_radius/3}" h="${wheel_width}"/>
     </link>
-    <link name= "${prefix}_${suffix}_wheel1">
+    <link name= "${prefix}_wheel1">
       <visual>
         <origin rpy= "0  ${PI/2} 0" xyz= "0 0 0"/>
         <geometry>
-          <mesh filename="package://robopi/meshes/tyre11.dae"/>
+          <mesh filename="package://bot_description/meshes/tyre11.dae"/>
         </geometry>
         <material name= "Black"/>
@@ -45,35 +46,12 @@
         <origin rpy= "0 ${PI/2} 0" xyz= "0 0 0"/>
         <geometry>
-          <mesh filename="package://robopi/meshes/tyre11.dae"/>
+          <mesh filename="package://bot_description/meshes/tyre11.dae"/>
         </geometry>
       </collision>
       <xacro:cylinder_inertia m="${wheel_mass}" r="${wheel_radius}" h="${wheel_width}"/>
     </link>
-    <joint name="${prefix}_${suffix}_wheel_joint1" type= "fixed">
-      <parent link="${prefix}_${suffix}_wheel"/>
-      <child link= "${prefix}_${suffix}_wheel1"/>
-      <origin xyz="0 0 0" rpy="0 0 0"/>
-    </joint>
-    <joint name="${prefix}_${suffix}_wheel_joint" type="continuous">
-      <parent link= "base_link"/>
-      <child link= "${prefix}_${suffix}_wheel"/>
-      <origin xyz= "${0.062*X-0.058*Y} ${(chassis_len/2+0.02)*Z}  0.015" rpy="0 0 0"/>
-      <axis xyz="0 1 0"/>
-      <limit effort= "100" velocity="100"/>
-      <dynamics damping="0.0" friction="0.0"/>
-    </joint>
-    <transmission name="${prefix}_${suffix}_wheel_trans">
-      <type>transmission_interface/SimpleTransmission</type>
-      <actuator name="${prefix}_${suffix}_wheel_motor">
-        <hardwareInterface>EffortJointInterface</hardwareInterface>
-        <mechanicalReduction>1</mechanicalReduction>
-      </actuator>
-      <joint name="${prefix}_${suffix}_wheel_joint">
-        <hardwareInterface>VelocityJointInterface</hardwareInterface>
-      </joint>
-    </transmission>
   </xacro:macro>
-  <xacro:wheel prefix="right" suffix="" X="0" Y="1" Z="-1"/>
-  <xacro:wheel prefix="left" suffix="" X="0" Y="1" Z="1"/>
+  <xacro:wheel prefix="right" X="0" Y="1" Z="-1"/>
+  <xacro:wheel prefix="left" X="0" Y="1" Z="1"/>
   <!-- <xacro:wheel prefix="right" suffix="front" X="1" Y="1" Z="-1"/>
      <xacro:wheel prefix="left" suffix="front" X="1" Y="1" Z="1"/>-->

File: bot_differential_drive/description/bot_differential_drive.ros2_control.xacro (robot description, xacro)
@@ -1,15 +1,23 @@
 <?xml version="1.0"?>
 <robot xmlns:xacro="http://www.ros.org/wiki/xacro">
-    <xacro:macro name="bot_ros2_control" params="name prefix">
+    <xacro:macro name="bot_ros2_control" params="name prefix use_mock_hardware">
         <ros2_control name="${name}" type="system">
-            <hardware>
-                <plugin>bot_differential_drive/DifferentialDriveSerialInterface</plugin>
-                <param name="left_wheel_name">left_wheel_joint</param>
-                <param name="right_wheel_name">right_wheel_joint</param>
-                <param name="loop_rate">100</param>
-                <param name="device_name">/dev/ttyACM0</param>
-                <param name="baud_rate">9600</param>
-                <param name="timeout_ms">1000</param>
-            </hardware>
+            <xacro:unless value="${use_mock_hardware}">
+                <hardware>
+                    <plugin>bot_differential_drive/DifferentialDriveSerialInterface</plugin>
+                    <param name="left_wheel_name">left_wheel_joint</param>
+                    <param name="right_wheel_name">right_wheel_joint</param>
+                    <param name="loop_rate">1000</param>
+                    <param name="device_name">/dev/ttyACM0</param>
+                    <param name="baud_rate">9600</param>
+                    <param name="timeout_ms">1000</param>
+                </hardware>
+            </xacro:unless>
+            <xacro:if value="${use_mock_hardware}">
+                <hardware>
+                    <plugin>mock_components/GenericSystem</plugin>
+                    <param name="calculate_dynamics">true</param>
+                </hardware>
+            </xacro:if>
             <joint name="${prefix}left_wheel_joint">
                 <command_interface name="velocity"/>

File: bot_differential_drive/description/bot_differential_drive.urdf.xacro (robot description, xacro)
@@ -5,6 +5,5 @@
   <xacro:arg name="use_mock_hardware" default="false" />
   <xacro:include filename="$(find bot_description)/urdf/bot.urdf.xacro" />
-  <!-- Import diffbot ros2_control description -->
   <xacro:include filename="$(find bot_differential_drive)/description/bot_differential_drive.ros2_control.xacro" />
-  <xacro:bot_ros2_control name="Bot" prefix="$(arg prefix)" />
+  <xacro:bot_ros2_control name="Bot" prefix="$(arg prefix)" use_mock_hardware="$(arg use_mock_hardware)" />
 </robot>
