Commit message: fix description lading / startup

File: bot_differential_drive/description/bot_differential_drive.ros2_control.xacro (robot description, xacro)
@@ -1,12 +1,12 @@
 <?xml version="1.0"?>
 <robot xmlns:xacro="http://www.ros.org/wiki/xacro">
-    <xacro:macro name="bot_control" params="name prefix">
+    <xacro:macro name="bot_ros2_control" params="name prefix">
         <ros2_control name="${name}" type="system">
             <hardware>
-                <plugin>diffdrive_arduino/DiffDriveArduinoHardware</plugin>
+                <plugin>bot_differential_drive/DifferentialDriveSerialInterface</plugin>
                 <param name="left_wheel_name">left_wheel_joint</param>
                 <param name="right_wheel_name">right_wheel_joint</param>
                 <param name="loop_rate">30</param>
-                <param name="device">/ttyACM0</param>
+                <param name="device_name">/dev/ttyACM0</param>
                 <param name="baud_rate">9600</param>
                 <param name="timeout_ms">1000</param>
