Commit message: - Removed: simulation related stuff - Changed: Naming of ros2 control files

File: bot_base/urdf/bot_base.urdf.xacro (robot description, xacro)
@@ -8,4 +8,4 @@
     <xacro:include filename="wheels.urdf.xacro" />
     <xacro:include filename="$(find bot_differential_drive)/description/bot_differential_drive.ros2_control.xacro" />
-    <xacro:bot_ros2_control name="Bot" prefix="$(arg prefix)" use_mock_hardware="$(arg use_mock_hardware)" />
+    <xacro:bot_differential_drive_control name="Bot" prefix="$(arg prefix)" use_mock_hardware="$(arg use_mock_hardware)" />
 </robot>

File: bot_differential_drive/description/bot_differential_drive.ros2_control.xacro (robot description, xacro)
@@ -1,5 +1,5 @@
 <?xml version="1.0"?>
 <robot xmlns:xacro="http://www.ros.org/wiki/xacro">
-    <xacro:macro name="bot_ros2_control" params="name prefix use_mock_hardware">
+    <xacro:macro name="bot_differential_drive_control" params="name prefix use_mock_hardware">
         <ros2_control name="${name}" type="system">
             <xacro:unless value="${use_mock_hardware}">
@@ -14,4 +14,5 @@
                 </hardware>
             </xacro:unless>
+            <!--
             <xacro:if value="${use_mock_hardware}">
                 <hardware>
@@ -25,5 +26,5 @@
                 </hardware>
             </xacro:if>
-            <!--
+            -->
             <xacro:if value="${use_mock_hardware}">
                 <hardware>
@@ -32,5 +33,4 @@
                 </hardware>
             </xacro:if>
-            -->
             <joint name="${prefix}left_wheel_joint">
                 <command_interface name="velocity"/>
