Commit message: Fixed: urdf and robot state publisher

File: bot_base/urdf/chassis.urdf.xacro (robot description, xacro)
@@ -1,3 +1,3 @@
-<robot name="robopi"
+<robot name="bot"
     xmlns:xacro="http://www.ros.org/wiki/xacro"
     xmlns:xi="http://www.w3.org/2001/XInclude">
@@ -9,5 +9,5 @@
             <origin rpy="-${PI/2} 0 ${PI/2}" xyz="0 0 0"/>
             <geometry>
-                <mesh filename="package://bot_description/meshes/base_assembly.dae"/>
+                <mesh filename="package://bot_base/meshes/base_assembly.dae"/>
             </geometry>
         </visual>
@@ -15,8 +15,8 @@
             <origin rpy="-${PI/2} 0 0" xyz="0 0 0"/>
             <geometry>
-                <mesh filename="package://bot_description/meshes/base_assembly.dae"/>
+                <mesh filename="package://bot_base/meshes/base_assembly.dae"/>
             </geometry>
         </collision>
-        <xacro:inertial_matrix mass="5.0"/>
+        <!--<xacro:inertial_matrix mass="5.0"/>-->
     </link>
     <!--///////////////////////////////////////////////////////////////// -->

File: bot_base/urdf/wheels.urdf.xacro (robot description, xacro)
@@ -7,17 +7,5 @@
   <xacro:property name="wheel_mass" value=".2"/>
   <xacro:macro name="wheel" params= "prefix X Y Z">
-    <joint name="${prefix}_wheel_joint1" type= "fixed">
-      <parent link="${prefix}_wheel"/>
-      <child link= "${prefix}_wheel1"/>
-      <origin xyz="0 0 0" rpy="0 0 0"/>
-    </joint>
-    <joint name="${prefix}_wheel_joint" type="continuous">
-      <parent link= "base_link"/>
-      <child link= "${prefix}_wheel"/>
-      <origin xyz= "${0.062*X-0.058*Y} ${(chassis_len/2+0.02)*Z}  0.015" rpy="0 0 0"/>
-      <axis xyz="0 1 0"/>
-      <dynamics damping="0.0" friction="0.0"/>
-    </joint>
-    <link name= "${prefix}_wheel">
+    <link name="${prefix}_wheel">
       <visual>
         <origin rpy= "${PI/2} 0 0" xyz= "0 0 0"/>
@@ -35,9 +23,9 @@
       <xacro:cylinder_inertia m="${wheel_mass}" r="${wheel_radius/3}" h="${wheel_width}"/>
     </link>
-    <link name= "${prefix}_wheel1">
+    <link name="${prefix}_wheel1">
       <visual>
         <origin rpy= "0  ${PI/2} 0" xyz= "0 0 0"/>
         <geometry>
-          <mesh filename="package://bot_description/meshes/tyre11.dae"/>
+          <mesh filename="package://bot_base/meshes/tyre11.dae"/>
         </geometry>
         <material name= "Black"/>
@@ -46,13 +34,23 @@
         <origin rpy= "0 ${PI/2} 0" xyz= "0 0 0"/>
         <geometry>
-          <mesh filename="package://bot_description/meshes/tyre11.dae"/>
+          <mesh filename="package://bot_base/meshes/tyre11.dae"/>
         </geometry>
       </collision>
       <xacro:cylinder_inertia m="${wheel_mass}" r="${wheel_radius}" h="${wheel_width}"/>
     </link>
+    <joint name="${prefix}_wheel_joint" type="fixed">
+      <parent link= "base_link"/>
+      <child link="${prefix}_wheel"/>
+      <origin xyz="${0.062*X-0.058*Y} ${(chassis_len/2+0.02)*Z}  0.015" rpy="0 0 0"/>
+      <axis xyz="0 1 0"/>
+      <dynamics damping="0.0" friction="0.0"/>
+    </joint>
+    <joint name="${prefix}_wheel_joint1" type= "fixed">
+      <parent link="${prefix}_wheel"/>
+      <child link="${prefix}_wheel1"/>
+      <origin xyz="0 0 0" rpy="0 0 0"/>
+    </joint>
   </xacro:macro>
-  <xacro:wheel prefix="right" X="0" Y="1" Z="-1"/>
-  <xacro:wheel prefix="left" X="0" Y="1" Z="1"/>
-  <!-- <xacro:wheel prefix="right" suffix="front" X="1" Y="1" Z="-1"/>
-     <xacro:wheel prefix="left" suffix="front" X="1" Y="1" Z="1"/>-->
+  <xacro:wheel prefix="right" X="1" Y="1" Z="-1"/>
+  <xacro:wheel prefix="left" X="1" Y="1" Z="1"/>
 </robot>

Commit message: update to simplified description which runs in gazebo

File: bot_base/urdf/chassis.urdf.xacro (robot description, xacro)
@@ -6,17 +6,22 @@
     <xacro:property name="chassis_height" value="0.070"/>
     <link name="base_link">
-        <visual>
-            <origin rpy="-${PI/2} 0 ${PI/2}" xyz="0 0 0"/>
+        <collision>
+            <origin xyz="-0.151427 -0 0.5" rpy="0 0 0"/>
             <geometry>
-                <mesh filename="package://bot_base/meshes/base_assembly.dae"/>
-            </geometry>
-        </visual>
-        <collision>
-            <origin rpy="-${PI/2} 0 0" xyz="0 0 0"/>
-            <geometry>
-                <mesh filename="package://bot_base/meshes/base_assembly.dae"/>
+                <box size="2.01142 1 0.568726"/>
             </geometry>
         </collision>
-        <!--<xacro:inertial_matrix mass="5.0"/>-->
+        <visual>
+            <origin xyz="-0.151427 -0 0.5" rpy="0 0 0"/>
+            <geometry>
+                <box size="2.01142 1 0.568726"/>
+            </geometry>
+            <material name="orange"/>
+        </visual>
+        <inertial>
+            <origin xyz="-0.151427 -0 0.5" rpy="0 0 0"/>
+            <mass value="1.14395"/>
+            <inertia ixx="0.126164" ixy="0.0" ixz="0.0" iyy="0.416519" iyz="0.0" izz="0.481014"/>
+        </inertial>
     </link>
     <!--///////////////////////////////////////////////////////////////// -->

File: bot_base/urdf/wheels.urdf.xacro (robot description, xacro)
@@ -6,51 +6,77 @@
   <xacro:property name="wheel_height" value="0.11"/>
   <xacro:property name="wheel_mass" value=".2"/>
-  <xacro:macro name="wheel" params= "prefix X Y Z">
-    <link name="${prefix}_wheel">
-      <visual>
-        <origin rpy= "${PI/2} 0 0" xyz= "0 0 0"/>
-        <geometry>
-          <cylinder length="${wheel_width}" radius= "${wheel_radius/5}"/>
-        </geometry>
-        <material name= "Black"/>
-      </visual>
-      <collision>
-        <origin rpy= "${PI/2} 0 0" xyz= "0 0 0"/>
-        <geometry>
-          <cylinder length="${wheel_width}" radius= "${wheel_radius/5}"/>
-        </geometry>
-      </collision>
-      <xacro:cylinder_inertia m="${wheel_mass}" r="${wheel_radius/3}" h="${wheel_width}"/>
-    </link>
-    <link name="${prefix}_wheel1">
-      <visual>
-        <origin rpy= "0  ${PI/2} 0" xyz= "0 0 0"/>
-        <geometry>
-          <mesh filename="package://bot_base/meshes/tyre11.dae"/>
-        </geometry>
-        <material name= "Black"/>
-      </visual>
-      <collision>
-        <origin rpy= "0 ${PI/2} 0" xyz= "0 0 0"/>
-        <geometry>
-          <mesh filename="package://bot_base/meshes/tyre11.dae"/>
-        </geometry>
-      </collision>
-      <xacro:cylinder_inertia m="${wheel_mass}" r="${wheel_radius}" h="${wheel_width}"/>
-    </link>
-    <joint name="${prefix}_wheel_joint" type="fixed">
-      <parent link= "base_link"/>
-      <child link="${prefix}_wheel"/>
-      <origin xyz="${0.062*X-0.058*Y} ${(chassis_len/2+0.02)*Z}  0.015" rpy="0 0 0"/>
-      <axis xyz="0 1 0"/>
-      <dynamics damping="0.0" friction="0.0"/>
-    </joint>
-    <joint name="${prefix}_wheel_joint1" type= "fixed">
-      <parent link="${prefix}_wheel"/>
-      <child link="${prefix}_wheel1"/>
-      <origin xyz="0 0 0" rpy="0 0 0"/>
-    </joint>
-  </xacro:macro>
-  <xacro:wheel prefix="right" X="1" Y="1" Z="-1"/>
-  <xacro:wheel prefix="left" X="1" Y="1" Z="1"/>
+  <joint name="left_wheel_joint" type="continuous">
+    <origin xyz="0.554283 0.625029 0.3" rpy="-1.5707 0 0"/>
+    <parent link="base_link"/>
+    <child link="left_wheel"/>
+    <axis xyz="0 0 1"/>
+    <dynamics damping="0.2"/>
+  </joint>
+  <!-- left wheel Link -->
+  <link name="left_wheel">
+    <collision>
+      <geometry>
+        <sphere radius="0.3"/>
+      </geometry>
+    </collision>
+    <visual>
+      <geometry>
+        <sphere radius="0.3"/>
+      </geometry>
+      <material name="black"/>
+    </visual>
+    <inertial>
+      <mass value="2"/>
+      <inertia ixx="0.145833" ixy="0.0" ixz="0.0" iyy="0.145833" iyz="0.0" izz="0.125"/>
+    </inertial>
+  </link>
+  <joint name="right_wheel_joint" type="continuous">
+    <origin xyz="0.554283 -0.625029 0.3" rpy="-1.5707 0 0"/>
+    <parent link="base_link"/>
+    <child link="right_wheel"/>
+    <axis xyz="0 0 1"/>
+    <dynamics damping="0.2"/>
+  </joint>
+  <!-- right wheel Link -->
+  <link name="right_wheel">
+    <collision>
+      <geometry>
+        <sphere radius="0.3"/>
+      </geometry>
+    </collision>
+    <visual>
+      <geometry>
+        <sphere radius="0.3"/>
+      </geometry>
+      <material name="black"/>
+    </visual>
+    <inertial>
+      <mass value="2"/>
+      <inertia ixx="0.145833" ixy="0.0" ixz="0.0" iyy="0.145833" iyz="0.0" izz="0.125"/>
+    </inertial>
+  </link>
+  <joint name="caster_joint" type="fixed">
+    <origin xyz="-0.957138 -0 0.2" rpy="0 0 0"/>
+    <parent link="base_link"/>
+    <child link="caster"/>
+  </joint>
+  <!-- caster frontal wheel Link -->
+  <link name="caster">
+    <collision>
+      <geometry>
+        <sphere radius="0.2"/>
+      </geometry>
+    </collision>
+    <visual>
+      <geometry>
+        <sphere radius="0.2"/>
+      </geometry>
+      <material name="white"/>
+    </visual>
+    <inertial>
+      <origin xyz="-0.957138 -0 0.2" rpy="0 0 0"/>
+      <mass value="0.005"/>
+      <inertia ixx="0.1" ixy="0.0" ixz="0.0" iyy="0.1" iyz="0.0" izz="0.1"/>
+    </inertial>
+  </link>
 </robot>
